Commit message: fix(t21): review findings - lio crash, TF loop, localizer yaw drift, IMU pose prediction
FastLIO2 frontend
- size the per-scan work buffers to the downsampled scan (fixed 10k buffers overflowed and
  segfaulted on the 2nd scan with airy.yaml's 5 cm voxel); point-selection flags no longer a
  vector<bool> written from an OpenMP loop; diagnostic counters are OMP reductions
- PointCloud2: drop NaN/Inf points; rebase per-point time on the EARLIEST point in double; with
  absolute per-point times the scan start comes from the points, not the header (rslidar_sdk
  ts_first_point=false stamps the last point)
- leg/wheel odometry is buffered and applied on the filter thread at the scan-end state, with the
  base->IMU extrinsic and w x r lever arm (it updated the IESKF from the sensor thread, racing it)
- IMU LPF off by default; when on, accel AND gyro share one filter (no relative skew), primed on
  the first sample, own sample-rate key; IMU filters reset after an IMU stream discontinuity
- IESKF covariance has a defined value before IMU init

Localization
- localizer: every rotation entering the outlier gate is projected onto SO(3); float ICP
  rounding compounded through the self-seeded tracker and the EMA turned it into a monotonic
  map->odom yaw creep (+0.7 deg / 100 s); prior map loaded at startup; update_hz 10;
  refine inlier gate 0.85 (measured: true pose >= 0.996, 0.5 m / 3 deg off <= 0.76);
  relocalize RPY composed in ZYX
- robot_pose: default odom_topic /mapping/lio_odom (production lio_node namespace); 20 Hz timer
  on the node clock; new imu_predict mode propagates the newest LIO state to the query time with
  the measured IMU samples (imu_propagation.hpp, own 0.25 s bound, all gates shared).  Gazebo,
  judged at the consumer's "now": 1.0 m/s 3D RMSE 1.3 cm / 98% post-lock output vs 9.8 cm for
  constant velocity.  Default on in universe.launch.py

TF / launch
- URDF root is `body` (the IMU frame lio_node estimates): odom -> body -> base_link -> sensors,
  body->base_link derived from the measured IMU mount; removes the extra body->base_link static
  TF that gave body two parents and closed a loop; mounts are launch args
- universe/sensing: robot_pose gets /mapping/lio_odom; unused rs_to_fastlio adapter not started;
  standalone localizer/pgo launches use the mapping namespace; max_prediction_s / imu_predict args
- rs_to_fastlio: NaN filtering, UINT16 ring, datatype-derived time scale, header = scan start

PGO
- offset read under the lock for TF; one worker thread (in-order keyframes); ExactTime sync;
  loop_enable_scan_context actually switches Scan Context
- built and run in Gazebo against fast_gicp 0e7ec14 (README build step pinned): correct
  rejection with no drift, 6 accepted loops and 0.75 -> 0.53 m RMSE under injected drift

Profiles / tools / tests
- airy.yaml / odin1.yaml: removed the MID360 extrinsic, the 1e-9 scale on a seconds field, the
  unsourced 18.5/37 Hz notch and the unbacked "Allan calibrated" noise; preflight now blocks
  them; fixture corrected
- test_t3_localization: predict mode must also pass the full-span availability gate
- new tests: dense-scan LidarProcessor, parser NaN/order/epoch, gate SO(3) drift, IMU LPF,
  IMU propagation (closed form) and the IMU predict path
- docs: correction notes on the synthetic "ALL PASS" report and the gait-filter premise; TF
  contract; Gazebo regression record docs/validation/gazebo_regression_20261018.md

Co-Authored-By: Claude Opus 5.5 (1M context) <noreply@anthropic.com>

File: src/description/quadruped_description/urdf/quadruped_sensors.urdf.xacro (robot description, xacro)
@@ -1,17 +1,32 @@
 <?xml version="1.0"?>
 <robot xmlns:xacro="http://www.ros.org/wiki/xacro" name="quadruped_robot">
-  <!-- Arguments for sensor mounting transforms -->
-  <xacro:property name="imu_x" value="-0.0110"/>
-  <xacro:property name="imu_y" value="-0.02329"/>
-  <xacro:property name="imu_z" value="0.04412"/>
-  <xacro:property name="imu_roll" value="0.0"/>
-  <xacro:property name="imu_pitch" value="0.0"/>
-  <xacro:property name="imu_yaw" value="0.0"/>
-  <xacro:property name="lidar_x" value="0.0"/>
-  <xacro:property name="lidar_y" value="0.0"/>
-  <xacro:property name="lidar_z" value="0.0"/>
-  <xacro:property name="lidar_roll" value="0.0"/>
-  <xacro:property name="lidar_pitch" value="0.0"/>
-  <xacro:property name="lidar_yaw" value="0.0"/>
+  <!-- Sensor mounts relative to base_link, MEASURED on the robot (calibration_procedure.md).
+       The defaults are placeholders, not a calibration.  imu_* is the IMU that FastLIO2 integrates;
+       ext_il in the lio yaml must equal T_imu<-lidar derived from these two mounts. -->
+  <xacro:arg name="imu_x" default="0.0"/>
+  <xacro:arg name="imu_y" default="0.0"/>
+  <xacro:arg name="imu_z" default="0.0"/>
+  <xacro:arg name="imu_roll" default="0.0"/>
+  <xacro:arg name="imu_pitch" default="0.0"/>
+  <xacro:arg name="imu_yaw" default="0.0"/>
+  <xacro:arg name="lidar_x" default="0.0"/>
+  <xacro:arg name="lidar_y" default="0.0"/>
+  <xacro:arg name="lidar_z" default="0.0"/>
+  <xacro:arg name="lidar_roll" default="0.0"/>
+  <xacro:arg name="lidar_pitch" default="0.0"/>
+  <xacro:arg name="lidar_yaw" default="0.0"/>
+  <!-- body -> base_link = inverse of the IMU mount; computed by rsp.launch.py from the imu_* args -->
+  <xacro:arg name="body_to_base_xyz" default="0 0 0"/>
+  <xacro:arg name="body_to_base_rpy" default="0 0 0"/>
+  <!-- TF tree root.  `body` is the frame FastLIO2 estimates (the IMU, odom -> body published by
+       lio_node), so it is the root here: odom -> body -> base_link -> sensors gives every frame
+       exactly ONE parent.  (A base_link -> body joint plus a body -> base_link static TF, as before,
+       made body a two-parent node and closed a loop.) -->
+  <link name="body"/>
+  <joint name="body_to_base_joint" type="fixed">
+    <parent link="body"/>
+    <child link="base_link"/>
+    <origin xyz="$(arg body_to_base_xyz)" rpy="$(arg body_to_base_rpy)"/>
+  </joint>
   <!-- Base link (REP-105 body center) -->
   <link name="base_link">
@@ -26,11 +41,4 @@
     </visual>
   </link>
-  <!-- Legacy body frame (coincident with base_link) -->
-  <link name="body"/>
-  <joint name="base_to_body_joint" type="fixed">
-    <parent link="base_link"/>
-    <child link="body"/>
-    <origin xyz="0 0 0" rpy="0 0 0"/>
-  </joint>
   <!-- IMU link -->
   <link name="imu_link">
@@ -48,5 +56,5 @@
     <parent link="base_link"/>
     <child link="imu_link"/>
-    <origin xyz="${imu_x} ${imu_y} ${imu_z}" rpy="${imu_roll} ${imu_pitch} ${imu_yaw}"/>
+    <origin xyz="$(arg imu_x) $(arg imu_y) $(arg imu_z)" rpy="$(arg imu_roll) $(arg imu_pitch) $(arg imu_yaw)"/>
   </joint>
   <!-- RoboSense Airy / Odin1 LiDAR link -->
@@ -65,12 +73,20 @@
     <parent link="base_link"/>
     <child link="lidar_link"/>
-    <origin xyz="${lidar_x} ${lidar_y} ${lidar_z}" rpy="${lidar_roll} ${lidar_pitch} ${lidar_yaw}"/>
+    <origin xyz="$(arg lidar_x) $(arg lidar_y) $(arg lidar_z)" rpy="$(arg lidar_roll) $(arg lidar_pitch) $(arg lidar_yaw)"/>
   </joint>
-  <!-- Camera link (for FastLIVO2 upgrade) -->
+  <!-- Camera link (FastLIVO2 upgrade).  camera_link is the OPTICAL frame (z forward, x right,
+       y down), so a forward-looking camera has rpy = (-pi/2, 0, -pi/2) relative to base_link.
+       Must agree with ext_lc (lidar -> camera) in the lio yaml; placeholder until calibrated. -->
+  <xacro:arg name="cam_x" default="0.0"/>
+  <xacro:arg name="cam_y" default="0.0"/>
+  <xacro:arg name="cam_z" default="0.0"/>
+  <xacro:arg name="cam_roll" default="-1.5707963"/>
+  <xacro:arg name="cam_pitch" default="0.0"/>
+  <xacro:arg name="cam_yaw" default="-1.5707963"/>
   <link name="camera_link"/>
   <joint name="base_to_camera_joint" type="fixed">
     <parent link="base_link"/>
     <child link="camera_link"/>
-    <origin xyz="0.055 -0.024 -0.036" rpy="0 0 0"/>
+    <origin xyz="$(arg cam_x) $(arg cam_y) $(arg cam_z)" rpy="$(arg cam_roll) $(arg cam_pitch) $(arg cam_yaw)"/>
   </joint>
 </robot>
